Commit message: Fix URDF includes that were pointing to original package

File: urdf/mech/base.urdf.xacro (robot description, xacro)
@@ -8,5 +8,5 @@
         <geometry>
           <!-- box size="${length} ${width} ${height}"/ -->
-          <mesh filename="package://linorobot2_description/meshes/elsabot_4wd.stl" scale="1.0 1.0 1.0"/> -->
+          <mesh filename="package://elsabot_4wd/meshes/elsabot_4wd.stl" scale="1.0 1.0 1.0"/> -->
         </geometry>
         <material name="gray">

File: urdf/robots/2wd.urdf.xacro (robot description, xacro)
@@ -1,12 +1,12 @@
 <?xml version="1.0"?>
-<robot name="linorobot2_2wd" xmlns:xacro="http://ros.org/wiki/xacro">
-  <xacro:include filename="$(find linorobot2_description)/urdf/2wd_properties.urdf.xacro" />
-  <xacro:include filename="$(find linorobot2_description)/urdf/mech/base.urdf.xacro" />
-  <xacro:include filename="$(find linorobot2_description)/urdf/mech/wheel.urdf.xacro" />
-  <xacro:include filename="$(find linorobot2_description)/urdf/mech/caster_wheel.urdf.xacro" />
-  <xacro:include filename="$(find linorobot2_description)/urdf/sensors/imu.urdf.xacro" />
-  <xacro:include filename="$(find linorobot2_description)/urdf/sensors/generic_laser.urdf.xacro" />
-  <xacro:include filename="$(find linorobot2_description)/urdf/sensors/depth_sensor.urdf.xacro" />
-  <xacro:include filename="$(find linorobot2_description)/urdf/controllers/diff_drive.urdf.xacro" />
+<robot name="elsabot_4wd" xmlns:xacro="http://ros.org/wiki/xacro">
+  <xacro:include filename="$(find elsabot_4wd)/urdf/2wd_properties.urdf.xacro" />
+  <xacro:include filename="$(find elsabot_4wd)/urdf/mech/base.urdf.xacro" />
+  <xacro:include filename="$(find elsabot_4wd)/urdf/mech/wheel.urdf.xacro" />
+  <xacro:include filename="$(find elsabot_4wd)/urdf/mech/caster_wheel.urdf.xacro" />
+  <xacro:include filename="$(find elsabot_4wd)/urdf/sensors/imu.urdf.xacro" />
+  <xacro:include filename="$(find elsabot_4wd)/urdf/sensors/generic_laser.urdf.xacro" />
+  <xacro:include filename="$(find elsabot_4wd)/urdf/sensors/depth_sensor.urdf.xacro" />
+  <xacro:include filename="$(find elsabot_4wd)/urdf/controllers/diff_drive.urdf.xacro" />
   <xacro:base
     length="${base_length}"

File: urdf/robots/4wd.urdf.xacro (robot description, xacro)
@@ -1,12 +1,12 @@
 <?xml version="1.0"?>
-<robot name="linorobot2_2wd" xmlns:xacro="http://ros.org/wiki/xacro">
-  <xacro:include filename="$(find linorobot2_description)/urdf/4wd_properties.urdf.xacro" />
-  <xacro:include filename="$(find linorobot2_description)/urdf/mech/base.urdf.xacro" />
-  <xacro:include filename="$(find linorobot2_description)/urdf/mech/wheel.urdf.xacro" />
-  <xacro:include filename="$(find linorobot2_description)/urdf/sensors/imu.urdf.xacro" />
-  <xacro:include filename="$(find linorobot2_description)/urdf/sensors/generic_laser.urdf.xacro" />
-  <!--xacro:include filename="$(find linorobot2_description)/urdf/sensors/depth_sensor.urdf.xacro" /-->
-  <xacro:include filename="$(find linorobot2_description)/urdf/sensors/oakd_on_ptbase.urdf.xacro" />
-  <xacro:include filename="$(find linorobot2_description)/urdf/controllers/skid_steer.urdf.xacro" />
+<robot name="elsabot_4wd" xmlns:xacro="http://ros.org/wiki/xacro">
+  <xacro:include filename="$(find elsabot_4wd)/urdf/4wd_properties.urdf.xacro" />
+  <xacro:include filename="$(find elsabot_4wd)/urdf/mech/base.urdf.xacro" />
+  <xacro:include filename="$(find elsabot_4wd)/urdf/mech/wheel.urdf.xacro" />
+  <xacro:include filename="$(find elsabot_4wd)/urdf/sensors/imu.urdf.xacro" />
+  <xacro:include filename="$(find elsabot_4wd)/urdf/sensors/generic_laser.urdf.xacro" />
+  <!--xacro:include filename="$(find elsabot_4wd)/urdf/sensors/depth_sensor.urdf.xacro" /-->
+  <xacro:include filename="$(find elsabot_4wd)/urdf/sensors/oakd_on_ptbase.urdf.xacro" />
+  <xacro:include filename="$(find elsabot_4wd)/urdf/controllers/skid_steer.urdf.xacro" />
   <xacro:base
     length="${base_length}"

File: urdf/robots/mecanum.urdf.xacro (robot description, xacro)
@@ -1,11 +1,11 @@
 <?xml version="1.0"?>
-<robot name="linorobot2_2wd" xmlns:xacro="http://ros.org/wiki/xacro">
-  <xacro:include filename="$(find linorobot2_description)/urdf/mecanum_properties.urdf.xacro" />
-  <xacro:include filename="$(find linorobot2_description)/urdf/mech/base.urdf.xacro" />
-  <xacro:include filename="$(find linorobot2_description)/urdf/mech/mecanum_wheel.urdf.xacro" />
-  <xacro:include filename="$(find linorobot2_description)/urdf/sensors/imu.urdf.xacro" />
-  <xacro:include filename="$(find linorobot2_description)/urdf/sensors/generic_laser.urdf.xacro" />
-  <xacro:include filename="$(find linorobot2_description)/urdf/sensors/depth_sensor.urdf.xacro" />
-  <xacro:include filename="$(find linorobot2_description)/urdf/controllers/omni_drive.urdf.xacro" />
+<robot name="elsabot_4wd" xmlns:xacro="http://ros.org/wiki/xacro">
+  <xacro:include filename="$(find elsabot_4wd)/urdf/mecanum_properties.urdf.xacro" />
+  <xacro:include filename="$(find elsabot_4wd)/urdf/mech/base.urdf.xacro" />
+  <xacro:include filename="$(find elsabot_4wd)/urdf/mech/mecanum_wheel.urdf.xacro" />
+  <xacro:include filename="$(find elsabot_4wd)/urdf/sensors/imu.urdf.xacro" />
+  <xacro:include filename="$(find elsabot_4wd)/urdf/sensors/generic_laser.urdf.xacro" />
+  <xacro:include filename="$(find elsabot_4wd)/urdf/sensors/depth_sensor.urdf.xacro" />
+  <xacro:include filename="$(find elsabot_4wd)/urdf/controllers/omni_drive.urdf.xacro" />
   <xacro:base
     length="${base_length}"

File: urdf/robots/square.urdf.xacro (robot description, xacro)
@@ -1,4 +1,4 @@
 <?xml version="1.0"?>
-<robot name="linorobot2_2wd" xmlns:xacro="http://ros.org/wiki/xacro">
+<robot name="elsabot_4wd" xmlns:xacro="http://ros.org/wiki/xacro">
   <xacro:property name="base_length" value="0.25" />
   <xacro:property name="base_width" value="0.25" />
@@ -14,11 +14,11 @@
   <xacro:property name="front_caster_wheel" value="false" />
   <xacro:property name="rear_caster_wheel" value="true" />
-  <xacro:include filename="$(find linorobot2_description)/urdf/mech/base.urdf.xacro" />
-  <xacro:include filename="$(find linorobot2_description)/urdf/mech/wheel.urdf.xacro" />
-  <xacro:include filename="$(find linorobot2_description)/urdf/mech/caster_wheel.urdf.xacro" />
-  <xacro:include filename="$(find linorobot2_description)/urdf/sensors/imu.urdf.xacro" />
-  <xacro:include filename="$(find linorobot2_description)/urdf/sensors/generic_laser.urdf.xacro" />
-  <xacro:include filename="$(find linorobot2_description)/urdf/sensors/depth_sensor.urdf.xacro" />
-  <xacro:include filename="$(find linorobot2_description)/urdf/controllers/diff_drive.urdf.xacro" />
+  <xacro:include filename="$(find elsabot_4wd)/urdf/mech/base.urdf.xacro" />
+  <xacro:include filename="$(find elsabot_4wd)/urdf/mech/wheel.urdf.xacro" />
+  <xacro:include filename="$(find elsabot_4wd)/urdf/mech/caster_wheel.urdf.xacro" />
+  <xacro:include filename="$(find elsabot_4wd)/urdf/sensors/imu.urdf.xacro" />
+  <xacro:include filename="$(find elsabot_4wd)/urdf/sensors/generic_laser.urdf.xacro" />
+  <xacro:include filename="$(find elsabot_4wd)/urdf/sensors/depth_sensor.urdf.xacro" />
+  <xacro:include filename="$(find elsabot_4wd)/urdf/controllers/diff_drive.urdf.xacro" />
   <xacro:property name="laser_pose">
     <origin xyz="0.0 0 0.325" rpy="-3.1416 0 0"/>

File: urdf/sensors/generic_laser.urdf.xacro (robot description, xacro)
@@ -1,5 +1,5 @@
 <?xml version="1.0"?>
 <robot xmlns:xacro="http://ros.org/wiki/xacro">
-  <xacro:include filename="$(find linorobot2_description)/urdf/sensors/laser.urdf.xacro" />
+  <xacro:include filename="$(find elsabot_4wd)/urdf/sensors/laser.urdf.xacro" />
   <xacro:macro name="generic_laser" params="*origin">
     <xacro:laser

File: urdf/sensors/oakd_on_ptbase.urdf.xacro (robot description, xacro)
@@ -79,5 +79,5 @@
         <geometry>
           <!-- box size="${length} ${width} ${height}"/ -->
-          <mesh filename="package://linorobot2_description/meshes/oakd.stl" scale="1.0 1.0 1.0"/> -->
+          <mesh filename="package://elsabot_4wd/meshes/oakd.stl" scale="1.0 1.0 1.0"/> -->
         </geometry>
         <material name="black">
