Commit message: Update to Humble and add Gazebo Ign support (WIP)
Gazebo functionality:
1. Robot appears in sim world.
2. Teleop moves it.
3. Nav will move it.

 Issues:
*  Localization not working.

File: urdf/controllers/diff_drive.urdf.xacro (robot description, xacro)
@@ -2,19 +2,24 @@
   <xacro:macro name="diff_drive_controller" params="wheel_separation wheel_radius wheel_torque">
     <gazebo>
-      <plugin name="differential_drive_controller" filename="libgazebo_ros_diff_drive.so">
-        <ros>
-          <argument>odom:=odom/unfiltered</argument>
-        </ros>
-        <updateRate>100</updateRate>
+      <plugin
+        filename="ignition-gazebo-diff-drive-system"
+        name="ignition::gazebo::systems::DiffDrive">
         <left_joint>left_wheel_joint</left_joint>
         <right_joint>right_wheel_joint</right_joint>
         <wheel_separation>${wheel_separation}</wheel_separation>
-        <wheel_diameter>${wheel_radius * 2}</wheel_diameter>
-        <max_wheel_acceleration>1.0</max_wheel_acceleration>
-        <robot_base_frame>base_footprint</robot_base_frame>
-        <publish_odom>true</publish_odom>
-        <publish_odom_tf>false</publish_odom_tf>
-        <publish_wheel_tf>true</publish_wheel_tf>
-        <odometry_frame>odom</odometry_frame>
+        <wheel_radius>${wheel_radius * 2}</wheel_radius>
+        <max_linear_acceleration>1</max_linear_acceleration>
+        <min_linear_acceleration>-1</min_linear_acceleration>
+        <max_angular_acceleration>2</max_angular_acceleration>
+        <min_angular_acceleration>-2</min_angular_acceleration>
+        <max_linear_velocity>0.5</max_linear_velocity>
+        <min_linear_velocity>-0.5</min_linear_velocity>
+        <max_angular_velocity>1</max_angular_velocity>
+        <min_angular_velocity>-1</min_angular_velocity>
+        <topic>cmd_vel</topic>
+        <odom_topic>odom</odom_topic>
+        <odom_publish_frequency>20</odom_publish_frequency>
+        <frame_id>odom</frame_id>
+        <child_frame_id>base_footprint</child_frame_id>
       </plugin>
     </gazebo>

File: urdf/controllers/skid_steer.urdf.xacro (robot description, xacro)
@@ -2,9 +2,7 @@
   <xacro:macro name="diff_drive_controller" params="wheel_separation wheel_radius wheel_torque">
     <gazebo>
-      <plugin name="differential_drive_controller" filename="libgazebo_ros_diff_drive.so">
-        <ros>
-          <argument>odom:=odom/unfiltered</argument>
-        </ros>
-        <num_wheel_pairs>2</num_wheel_pairs>
+      <plugin
+        filename="ignition-gazebo-diff-drive-system"
+        name="ignition::gazebo::systems::DiffDrive">
         <left_joint>front_left_wheel_joint</left_joint>
         <right_joint>front_right_wheel_joint</right_joint>
@@ -12,14 +10,18 @@
         <right_joint>rear_right_wheel_joint</right_joint>
         <wheel_separation>${wheel_separation}</wheel_separation>
-        <wheel_separation>${wheel_separation}</wheel_separation>
-        <wheel_diameter>${wheel_radius * 2}</wheel_diameter>
-        <wheel_diameter>${wheel_radius * 2}</wheel_diameter>
-        <updateRate>100</updateRate>
-        <max_wheel_acceleration>1.0</max_wheel_acceleration>
-        <robot_base_frame>base_footprint</robot_base_frame>
-        <publish_odom>true</publish_odom>
-        <publish_odom_tf>false</publish_odom_tf>
-        <publish_wheel_tf>true</publish_wheel_tf>
-        <odometry_frame>odom</odometry_frame>
+        <wheel_radius>${wheel_radius * 2}</wheel_radius>
+        <max_linear_acceleration>1</max_linear_acceleration>
+        <min_linear_acceleration>-1</min_linear_acceleration>
+        <max_angular_acceleration>2</max_angular_acceleration>
+        <min_angular_acceleration>-2</min_angular_acceleration>
+        <max_linear_velocity>0.5</max_linear_velocity>
+        <min_linear_velocity>-0.5</min_linear_velocity>
+        <max_angular_velocity>1</max_angular_velocity>
+        <min_angular_velocity>-1</min_angular_velocity>
+        <topic>cmd_vel</topic>
+        <odom_topic>odom</odom_topic>
+        <odom_publish_frequency>20</odom_publish_frequency>
+        <frame_id>odom</frame_id>
+        <child_frame_id>base_footprint</child_frame_id>
       </plugin>
     </gazebo>

File: urdf/mech/base.urdf.xacro (robot description, xacro)
@@ -8,5 +8,5 @@
         <geometry>
           <!-- box size="${length} ${width} ${height}"/ -->
-          <mesh filename="package://elsabot_4wd/meshes/elsabot_4wd.stl" scale="1.0 1.0 1.0"/> -->
+          <mesh filename="package://elsabot_4wd/meshes/elsabot_4wd.stl" scale="1.0 1.0 1.0"/>
         </geometry>
         <material name="gray">

File: urdf/mech/wheel.urdf.xacro (robot description, xacro)
@@ -33,4 +33,6 @@
       <origin xyz="${pos_x} ${pos_y} ${pos_z}" rpy="0 0 0"/>
     </joint>
+    <gazebo reference="${side}_wheel_joint">
+    </gazebo>
   </xacro:macro>
 </robot>

File: urdf/robots/4wd.urdf.xacro (robot description, xacro)
@@ -60,4 +60,12 @@
     <xacro:insert_block name="depth_sensor_pose" />
   </xacro:depth_sensor>
+  <gazebo>
+    <plugin filename="ignition-gazebo-joint-state-publisher-system" name="ignition::gazebo::systems::JointStatePublisher"/>
+    <plugin filename="ignition-gazebo-sensors-system" name="ignition::gazebo::systems::Sensors">
+      <render_engine>ogre2</render_engine>
+    </plugin>
+    <plugin filename="ignition-gazebo-imu-system" name="ignition::gazebo::systems::Imu">
+    </plugin>
+  </gazebo>
   <xacro:diff_drive_controller
     wheel_separation="${wheel_pos_y * 2}"

File: urdf/sensors/imu.urdf.xacro (robot description, xacro)
@@ -1,5 +1,13 @@
 <robot xmlns:xacro="http://ros.org/wiki/xacro">
   <xacro:macro name="imu">
-    <link name="imu_link"/>
+    <link name="imu_link">
+      <inertial>
+        <origin xyz="0 0 0" rpy="0 0 0"/>
+        <mass value="0.1"/>
+        <inertia ixx="0.1" ixy="0" ixz="0"
+                 iyy="0.1" iyz="0"
+                 izz="0.1" />
+      </inertial>
+    </link>
     <joint name="imu_to_base_link" type="fixed">
       <parent link="base_link"/>
@@ -9,23 +17,15 @@
     <gazebo reference="imu_link">
       <gravity>true</gravity>
-      <sensor name="imu_sensor" type="imu">
-      <always_on>true</always_on>
+      <sensor name="imu_link" type="imu">
+        <topic>imu/data</topic>
+        <frameName>imu_link</frameName>
+        <ignition_frame_id>imu_link</ignition_frame_id>
+        <always_on>1</always_on>
       <update_rate>20</update_rate>
       <visualize>true</visualize>
-      <topic>__default_topic__</topic>
-      <plugin filename="libgazebo_ros_imu_sensor.so" name="imu_plugin">
-          <ros>
-            <remapping>~/out:=imu/data</remapping>
-          </ros>
-          <topicName>imu/data</topicName>
-          <bodyName>imu_link</bodyName>
-          <updateRateHZ>10.0</updateRateHZ>
-          <gaussianNoise>0.0</gaussianNoise>
+        <gaussianNoise>0</gaussianNoise>
           <xyzOffset>0 0 0</xyzOffset>
           <rpyOffset>0 0 0</rpyOffset>
-          <frameName>imu_link</frameName>
           <initialOrientationAsReference>false</initialOrientationAsReference>
-      </plugin>
-      <pose>0 0 0 0 0 0</pose>
       </sensor>
     </gazebo>

File: urdf/sensors/laser.urdf.xacro (robot description, xacro)
@@ -42,10 +42,9 @@
     </joint>
     <gazebo reference="${frame_id}">
-      <sensor type="ray" name="${frame_id}_head_hokuyo_sensor">
-        <always_on>true</always_on>
-        <update_rate>${update_rate}</update_rate>
-        <pose>0 0 0 0 0 0</pose>
-        <visualize>false</visualize>
-        <ray>
+      <sensor name="${frame_id}" type='gpu_lidar'>
+        <topic>${topic_name}</topic>
+        <ignition_frame_id>${frame_id}</ignition_frame_id>
+        <update_rate>10</update_rate>
+        <lidar>
           <scan>
             <horizontal>
@@ -55,4 +54,10 @@
               <max_angle>${max_angle}</max_angle>
             </horizontal>
+            <vertical>
+              <samples>1</samples>
+              <resolution>0.01</resolution>
+              <min_angle>0.0</min_angle>
+              <max_angle>0.0</max_angle>
+            </vertical>
           </scan>
           <range>
@@ -61,16 +66,7 @@
             <resolution>0.01</resolution>
           </range>
-        </ray>
-        <plugin name="${frame_id}_gazebo_ros_head_hokuyo_controller" filename="libgazebo_ros_ray_sensor.so">
-          <ros>
-            <remapping>~/out:=${topic_name}</remapping>
-          </ros>
-          <output_type>sensor_msgs/LaserScan</output_type>
-          <alwaysOn>true</alwaysOn>
-          <updateRate>${update_rate}</updateRate>
-          <topicName>${topic_name}</topicName>
-          <frame_name>${frame_id}</frame_name>
-          <output_type>sensor_msgs/LaserScan</output_type>
-        </plugin>
+        </lidar>
+        <alwaysOn>1</alwaysOn>
+        <visualize>true</visualize>
       </sensor>
     </gazebo>

File: urdf/sensors/oakd_on_ptbase.urdf.xacro (robot description, xacro)
@@ -79,5 +79,5 @@
         <geometry>
           <!-- box size="${length} ${width} ${height}"/ -->
-          <mesh filename="package://elsabot_4wd/meshes/oakd.stl" scale="1.0 1.0 1.0"/> -->
+          <mesh filename="package://elsabot_4wd/meshes/oakd.stl" scale="1.0 1.0 1.0"/>
         </geometry>
         <material name="black">
