Commit message: Update position of GPS antenna for new mount

File: urdf/sensors/gps.urdf.xacro (robot description, xacro)
@@ -13,5 +13,5 @@
       <parent link="base_link"/>
       <child link="gps_link"/>
-      <origin xyz="-0.150 0.0 0.100" rpy="0 0 0"/>
+      <origin xyz="-0.195 0.0 0.685" rpy="0 0 0" />
     </joint>
     <gazebo reference="gps_link">
