Commit message: Support change in wheel position

File: urdf/4wd_properties.urdf.xacro (robot description, xacro)
@@ -7,5 +7,5 @@
   <xacro:property name="wheel_radius" value="0.0795" />
   <xacro:property name="wheel_width" value="0.047" />
-  <xacro:property name="wheel_pos_x" value="0.1505" />
+  <xacro:property name="wheel_pos_x" value="0.175" />
   <xacro:property name="wheel_pos_y" value="0.1925" />
   <xacro:property name="wheel_pos_z" value="-0.1105" />

Commit message: Gazebo changes

File: urdf/4wd_properties.urdf.xacro (robot description, xacro)
@@ -10,5 +10,5 @@
   <xacro:property name="wheel_pos_y" value="0.1925" />
   <xacro:property name="wheel_pos_z" value="-0.1105" />
-  <xacro:property name="wheel_mass" value=".6" />
+  <xacro:property name="wheel_mass" value="0.6" />
   <xacro:property name="wheel_torque" value="12" />
   <xacro:property name="laser_pose">

File: urdf/controllers/diff_drive.urdf.xacro (robot description, xacro)
@@ -23,4 +23,9 @@
         <child_frame_id>base_footprint</child_frame_id>
       </plugin>
+      <plugin filename="gz-sim-joint-state-publisher-system" name="gz::sim::systems::JointStatePublisher">
+        <joint_name>left_wheel_joint</joint_name>
+        <joint_name>front_right_wheel_joint</joint_name>
+        <topic>/joint_states</topic>
+      </plugin>
     </gazebo>
   </xacro:macro>

File: urdf/controllers/skid_steer.urdf.xacro (robot description, xacro)
@@ -25,4 +25,11 @@
         <child_frame_id>base_footprint</child_frame_id>
       </plugin>
+      <plugin filename="gz-sim-joint-state-publisher-system" name="gz::sim::systems::JointStatePublisher">
+        <joint_name>front_left_wheel_joint</joint_name>
+        <joint_name>front_right_wheel_joint</joint_name>
+        <joint_name>rear_left_wheel_joint</joint_name>
+        <joint_name>rear_right_wheel_joint</joint_name>
+        <topic>/joint_states</topic>
+      </plugin>
     </gazebo>
   </xacro:macro>

File: urdf/mech/wheel.urdf.xacro (robot description, xacro)
@@ -9,4 +9,21 @@
         </geometry>
       </collision>
+      <!--visual>
+        <origin xyz="0 0 0" rpy="${pi/2} 0 0"/>
+        <geometry>
+          <cylinder radius="${radius}" length="${width}"/>
+        </geometry>
+        <material name="black">
+            <color rgba="0.0 0.0 0.0 1.0"/>
+        </material>
+      </visual-->
+      <surface>
+        <friction>
+          <ode>
+            <mu>0.8</mu>
+            <mu2>0.8</mu2>
+          </ode>
+        </friction>
+      </surface>
       <inertial>
         <origin xyz="0 0 0" rpy="0 0 0"/>

File: urdf/robots/4wd.urdf.xacro (robot description, xacro)
@@ -10,4 +10,5 @@
   <xacro:include filename="$(find elsabot_4wd)/urdf/sensors/oakd_on_ptbase.urdf.xacro" />
   <xacro:include filename="$(find elsabot_4wd)/urdf/controllers/skid_steer.urdf.xacro" />
+  <xacro:include filename="$(find elsabot_4wd)/urdf/sensors/nav_camera.urdf.xacro" />
   <xacro:base
     length="${base_length}"
@@ -62,4 +63,5 @@
     <xacro:insert_block name="depth_sensor_pose" />
   </xacro:depth_sensor>
+  <xacro:nav_camera/>
  <xacro:diff_drive_controller
     wheel_separation="${wheel_pos_y * 2}"
@@ -68,5 +70,4 @@
   />
   <gazebo>
-    <plugin filename="gz-sim-joint-state-publisher-system" name="gz::sim::systems::JointStatePublisher"/>
     <plugin filename="gz-sim-sensors-system" name="gz::sim::systems::Sensors">
       <render_engine>ogre2</render_engine>

File: urdf/sensors/gps.urdf.xacro (robot description, xacro)
@@ -20,5 +20,5 @@
         <update_rate>2</update_rate>
         <topic>navsat</topic>
-        <ignition_frame_id>gps_link</ignition_frame_id>
+        <gz_frame_id>gps_link</gz_frame_id>
       </sensor>
     </gazebo>

File: urdf/sensors/imu.urdf.xacro (robot description, xacro)
@@ -13,5 +13,5 @@
       <parent link="base_link"/>
       <child link="imu_link"/>
-      <origin xyz="0 0.025 0.028" rpy="0 0 0"/>
+      <origin xyz="0.25 0.0 0.210" rpy="0 0 0"/>
     </joint>
     <gazebo reference="imu_link">
@@ -19,8 +19,8 @@
       <sensor name="imu_link" type="imu">
         <topic>imu/data</topic>
-        <ignition_frame_id>imu_link</ignition_frame_id>
+        <gz_frame_id>imu_link</gz_frame_id>
         <always_on>1</always_on>
-        <update_rate>10</update_rate>
-      	<visualize>true</visualize>
+        <update_rate>20</update_rate>
+        <visualize>true</visualize>
         <gaussianNoise>0</gaussianNoise>
         <xyzOffset>0 0 0</xyzOffset>
@@ -30,8 +30,8 @@
       <sensor name="magnetometer" type="magnetometer">
         <always_on>1</always_on>
-        <update_rate>10</update_rate>
+        <update_rate>20</update_rate>
         <visualize>true</visualize>
         <topic>imu/mag</topic>
-        <ignition_frame_id>imu_link</ignition_frame_id>
+        <gz_frame_id>imu_link</gz_frame_id>
         <enable_metrics>true</enable_metrics>
         <magnetometer>

File: urdf/sensors/laser.urdf.xacro (robot description, xacro)
@@ -44,5 +44,5 @@
       <sensor name="${frame_id}" type='gpu_lidar'>
         <topic>${topic_name}</topic>
-        <ignition_frame_id>${frame_id}</ignition_frame_id>
+        <gz_frame_id>${frame_id}</gz_frame_id>
         <update_rate>10</update_rate>
         <lidar>

File: urdf/sensors/oakd_on_ptbase.urdf.xacro (robot description, xacro)
@@ -106,4 +106,23 @@
       <child link="oakd_right_camera" />
     </joint>
+    <!-- https://github.com/ros-simulation/gazebo_ros_pkgs/wiki/ROS-2-Migration:-Camera#gazebo_ros_camera -->
+    <!--gazebo reference="oakd_center_camera">
+      <sensor name="camera" type="camera">
+        <always_on>true</always_on>
+        <update_rate>10.0</update_rate>
+        <gz_frame_id>camera_link_optical</gz_frame_id>
+        <topic>camera/image</topic>
+        <horizontal_fov>1.50098</horizontal_fov>
+        <image>
+            <width>640</width>
+            <height>480</height>
+            <format>R8G8B8</format>
+        </image>
+        <clip>
+            <near>0.02</near>
+            <far>300</far>
+        </clip>
+      </sensor>
+    </gazebo-->
   </xacro:macro>
 </robot>
